File: kicad/all-in-one-sensor/all-in-one-sensor.kicad_sch (KiCad schematic)
At the start: 17 parts, among them J2 BH170 (0x23), J3 mmWave, J4 mmWave2, U1 EKMC1603111, U2 BME280, U3 BME680, U4 WEMOS C3/D1 Mini

Commit message: closes #3: m3 mounting holes
Parts:
- H1, H2, H3, H4: footprint MountingHole:MountingHole_2.2mm_M2 -> MountingHole:MountingHole_3.2mm_M3
Changed lines of the file:
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@@
       (effects (font (size 1.27 1.27)) (justify left))
     )
-    (property "Footprint" "MountingHole:MountingHole_2.2mm_M2" (id 2) (at 258.572 33.02 0)
+    (property "Footprint" "MountingHole:MountingHole_3.2mm_M3" (id 2) (at 258.572 33.02 0)
       (effects (font (size 1.27 1.27)) hide)
     )
@@
       (effects (font (size 1.27 1.27)) (justify left))
     )
-    (property "Footprint" "MountingHole:MountingHole_2.2mm_M2" (id 2) (at 258.572 38.354 0)
+    (property "Footprint" "MountingHole:MountingHole_3.2mm_M3" (id 2) (at 258.572 38.354 0)
       (effects (font (size 1.27 1.27)) hide)
     )
@@
       (effects (font (size 1.27 1.27)) (justify left))
     )
-    (property "Footprint" "MountingHole:MountingHole_2.2mm_M2" (id 2) (at 258.572 43.688 0)
+    (property "Footprint" "MountingHole:MountingHole_3.2mm_M3" (id 2) (at 258.572 43.688 0)
       (effects (font (size 1.27 1.27)) hide)
     )
@@
       (effects (font (size 1.27 1.27)) (justify left))
     )
-    (property "Footprint" "MountingHole:MountingHole_2.2mm_M2" (id 2) (at 258.572 27.686 0)
+    (property "Footprint" "MountingHole:MountingHole_3.2mm_M3" (id 2) (at 258.572 27.686 0)
       (effects (font (size 1.27 1.27)) hide)
     )
@@
     )
     (path "/e06dc752-5808-4e2f-a147-d61d676e26c7"
-      (reference "H1") (unit 1) (value "MountingHole") (footprint "MountingHole:MountingHole_2.2mm_M2")
+      (reference "H1") (unit 1) (value "MountingHole") (footprint "MountingHole:MountingHole_3.2mm_M3")
     )
     (path "/35c91e06-7c71-48df-afab-7497cd76314a"
-      (reference "H2") (unit 1) (value "MountingHole") (footprint "MountingHole:MountingHole_2.2mm_M2")
+      (reference "H2") (unit 1) (value "MountingHole") (footprint "MountingHole:MountingHole_3.2mm_M3")
     )
     (path "/5a8d0a97-c1a5-48fc-9c4c-ea9fc633b330"
-      (reference "H3") (unit 1) (value "MountingHole") (footprint "MountingHole:MountingHole_2.2mm_M2")
+      (reference "H3") (unit 1) (value "MountingHole") (footprint "MountingHole:MountingHole_3.2mm_M3")
     )
     (path "/e05d7c0e-c3a5-4bb6-876f-57489f095f41"
-      (reference "H4") (unit 1) (value "MountingHole") (footprint "MountingHole:MountingHole_2.2mm_M2")
+      (reference "H4") (unit 1) (value "MountingHole") (footprint "MountingHole:MountingHole_3.2mm_M3")
     )
     (path "/ca276387-2714-49d7-9b67-2727b4263616"
